File: Electronics/PCB/FC Control board 0.0/FC Control board 1.0.kicad_sch (KiCad schematic)
At the start: 33 parts, among them J1 USB_C_Receptacle_USB2.0, J2 Conn_01x04_Pin, J3 Conn_01x03_Pin, SW1 RESET, SW2 BOOT, SW3 SW_SPST, U1 ESP32-S3-WROOM-1-N8, U2 AZ1117-3.3, U4 AZ1117-5.0, U6 INA4181A3IPWR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

Commit message: FC control board V1.0
As ordered from JLC
Parts:
- removed C10: C_Small, Capacitor_SMD:C_0603_1608Metric, symbol Device:C_Small
- removed J2: Conn_01x04_Pin, Connector_PinSocket_2.54mm:PinSocket_1x04_P2.54mm_Vertical, symbol Connector:Conn_01x04_Pin
- removed J3: Conn_01x03_Pin, Connector_PinSocket_2.54mm:PinSocket_1x03_P2.54mm_Vertical, symbol Connector:Conn_01x03_Pin
- removed JP1: SolderJumper_3_Bridged12, Jumper:SolderJumper-3_P1.3mm_Bridged12_RoundedPad1.0x1.5mm, symbol Jumper:SolderJumper_3_Bridged12
- removed R5, R6: R_Small, Resistor_SMD:R_0603_1608Metric_Pad0.98x0.95mm_HandSolder, symbol Device:R_Small
- removed RV1: R_Potentiometer_Small, Potentiometer_THT:Potentiometer_Alps_RK163_Single_Horizontal, symbol Device:R_Potentiometer_Small
- removed U6: INA4181A3IPWR, FC_footprint_library:SOP65P640X120-20N, symbol INA4181A3IPWR:INA4181A3IPWR
- removed U9: LM358_DFN, Package_SO:SOIC-8-1EP_3.9x4.9mm_P1.27mm_EP2.514x3.2mm, symbol Amplifier_Operational:LM358_DFN
- added BZ1: Buzzer1, Buzzer_Beeper:Buzzer_12x9.5RM7.6, symbol Device:Buzzer
- added BZ2: Buzzer2, Buzzer_Beeper:Buzzer_12x9.5RM7.6, symbol Device:Buzzer
- added BZ3: Buzzer3, Buzzer_Beeper:Buzzer_12x9.5RM7.6, symbol Device:Buzzer
- added C9: 10u, symbol Device:C
- added M2: Motor_DC_ALT, symbol Motor:Motor_DC_ALT
- added R10, R12, R5, R7: 5k, symbol Device:R
- added R11, R6, R8, R9: 10k, symbol Device:R
- added U4: NRF24L01_Breakout, RF_Module:nRF24L01_Breakout, symbol RF:NRF24L01_Breakout
- added U5: LM358DRG3 2_4, Package_SO:SOIC-8_3.9x4.9mm_P1.27mm, symbol Device:Opamp_Dual
- added U6: LM358DRG3 1_3, Package_SO:SOIC-8_3.9x4.9mm_P1.27mm, symbol Device:Opamp_Dual
- added U_M1: TB67H451AFNG,EL, Package_SO:HSOP-8-1EP_3.9x4.9mm_P1.27mm_EP2.41x3.1mm, symbol FC_library:TB67H451AFNG,EL
- added Volume1: R_Buzzer, Potentiometer_THT:Potentiometer_Alps_RK09K_Single_Horizontal, symbol Device:R_Potentiometer
- C1: footprint Capacitor_SMD:C_1206_3216Metric -> (none)
- R_bat1, R_bat2: footprint Resistor_SMD:R_0805_2012Metric_Pad1.20x1.40mm_HandSolder -> (none)
Connections:
- net M4_sense is gone; now on net bat_level: U1.4 (IO4)
- net +3V3: now also C9.2, U4.2 (VCC), Volume1.1, Volume1.2
- net GNDREF: now also BZ1.2 (+), BZ2.2 (+), BZ3.2 (+), C9.1, R11.2, R6.2, R8.2, R9.2, U4.1 (GND), U5.4 (V-), U6.4 (V-), U_M1.1 (GND)
- net MISO: now also U4.7 (MISO)
- net VCC: now also U5.8 (V+), U6.8 (V+), U_M1.5 (VM)
- net MOSI: now reaches U1.19 (IO11)
- net MOSI: now also U4.6 (MOSI)
- net SCK: now reaches U1.20 (IO12)
- net SCK: now also U4.5 (SCK)
- net ACD1_4 renamed CSN
- net CSN: now also U4.4 (~{CSN})
- net ACD1_5 renamed CE
- net CE: now also U4.3 (CE)
- net ACD1_6 renamed Volume_pot
- net Volume_pot: now also Volume1.3
- net ACD1_7 renamed SDA
- net ACD1_8 renamed bat_level
- net bat_level: no longer U1.17 (IO9)
- net ACD1_9 renamed SS
- net FWR_1 renamed M1_ref_3V
- net M1_ref_3V: now also U6.5 (+)
- net FWR_2 renamed M3_ref_3V
- net M3_ref_3V: now also U5.5 (+)
- net FWR_3: no longer names the net of U1.32 (IO39)
- net FWR_4: no longer names the net of U1.34 (IO41)
- net M1_sense: no longer names the net of U1.39 (IO1)
- net M2_sense: no longer names the net of U1.38 (IO2)
- net M3_sense: no longer names the net of U1.15 (IO3)
- net REV_1 renamed M2_ref_3V
- net M2_ref_3V: now also U5.3 (+)
- net REV_2 renamed M4_ref_3V
- net M4_ref_3V: now also U6.3 (+)
- net REV_3: no longer names the net of U1.33 (IO40)
- net REV_4: no longer names the net of U1.35 (IO42)
- new net: M2.1 (+), U_M1.8 (OUT2)
- new net: M2.2 (-), U_M1.6 (OUT1)
- new net: R7.2, R8.1, U5.2 (-)
- new net: R5.2, R6.1, U6.2 (-)
- new net: R11.1, R12.2, U5.6 (-)
- new net: R10.2, R9.1, U6.6 (-)
- new net BUZZER_PIN: BZ1.1 (-)
- new net BUZZER_PIN2: BZ2.1 (-)
- new net BUZZER_PIN3: BZ3.1 (-)
- new net M1_1: U_M1.2 (IN2)
- new net M1_2: U_M1.3 (IN1)
- new net M1_ref_5V: R10.1, U6.7
- new net M2_ref_5V: U5.1
- new net M3_ref_5V: R12.1, U5.7
- new net M4_ref_5V: R5.1, U6.1
- new net SCL: U1.17 (IO9)
- no-connect marks 19 -> 2
Other:
- removed sheet Motor driver
- removed sheet Motor driver1
- removed sheet Motor driver2
- removed sheet Motor driver3
- note added: "Reference signal boost from [0, 3.3]V to [0, 5.0]V"
- moved on the sheet: C1, U1
