File: Electronics/PCB/FC Control board 1.0/FC Control board 1.0.kicad_pcb (KiCad board)
At the start: 2 copper layers, 53.2 x 104.1 mm, 18 parts, among them J1 USB_C_Receptacle_USB2.0, SW1 RESET, SW2 BOOT, U1 ESP32-S3-WROOM-1-N8, U2 AZ1117-3.3, U3 TS321, U4 NRF24L01_Breakout

Commit message: Restart project
Parts:
- removed R_i-msr-M1: 1, Resistor_SMD:R_2512_6332Metric_Pad1.40x3.35mm_HandSolder
- added BZ1: Buzzer1, Buzzer_Beeper:Buzzer_12x9.5RM7.6, F.Cu at (126.4, 127.2)
- added BZ2: Buzzer2, Buzzer_Beeper:Buzzer_12x9.5RM7.6, F.Cu at (126.4, 140.7)
- added BZ3: Buzzer3, Buzzer_Beeper:Buzzer_12x9.5RM7.6, F.Cu at (126.4, 154.3)
- added C5: 10uF, Capacitor_SMD:C_1206_3216Metric, F.Cu at (139.8, 128.8)
- added C6: 10uF, Capacitor_SMD:C_1206_3216Metric, F.Cu at (139.8, 132.1)
- added C7: 10uF, Capacitor_SMD:C_1206_3216Metric, F.Cu at (139.8, 135.5)
- added C8: 10uF, Capacitor_SMD:C_1206_3216Metric, F.Cu at (139.8, 138.8)
- added U5: LM358DRG3 2_4, Package_SO:SOIC-8_3.9x4.9mm_P1.27mm, F.Cu at (146.9, 139.8)
- added U6: LM358DRG3 1_3, Package_SO:SOIC-8_3.9x4.9mm_P1.27mm, F.Cu at (146.9, 146.3)
- added U7: AZ1117-3.3, Package_TO_SOT_SMD:SOT-223-3_TabPin2, F.Cu at (156.0, 148.8)
- added Volume1: R_Buzzer, Potentiometer_THT:Potentiometer_Alps_RK09K_Single_Horizontal, F.Cu at (155.0, 126.0)
- BT1: footprint FC_footprint_library:1043_18650_Li-ion -> Connector_JST:JST_EH_B2B-EH-A_1x02_P2.50mm_Vertical; moved to F.Cu
- U3: value TS321 -> AZ1117-5.0; footprint Package_TO_SOT_SMD:SOT-23-5_HandSoldering -> Package_TO_SOT_SMD:TO-252-2
- moved U4 69.3 mm to (218.1, 169.5), turned to -90 degrees
- moved R1 61.0 mm to (145.0, 151.0)
- moved U3 55.8 mm to (158.0, 140.6)
- moved BT1 52.2 mm to (154.6, 155.5), turned to 0 degrees
- moved C3 43.3 mm to (139.8, 125.4)
- moved C2 38.3 mm to (139.8, 122.1)
- moved R2 25.2 mm to (218.1, 184.7)
- moved D1 16.2 mm to (207.7, 195.7)
- moved R3 13.1 mm to (210.4, 184.7), turned to 180 degrees
- moved SW1 4.40 mm to (195.9, 191.2), turned to -90 degrees
- moved SW2 2.70 mm to (203.2, 191.2), turned to -90 degrees
- moved J1 2.50 mm to (214.3, 193.3)
- moved U1 2.50 mm to (206.6, 151.7)
Connections:
- BT1 pad 2: GNDREF -> Net-(BT1--)
- U1 pad 12: unconnected-(U1-Pad12) -> /SDA
- U1 pad 13: unconnected-(U1-Pad13) -> /USB_D-
- U1 pad 14: unconnected-(U1-Pad14) -> /USB_D+
- U1 pad 17: unconnected-(U1-Pad17) -> /SCL
- U1 pad 18: unconnected-(U1-Pad18) -> /SS
- U1 pad 19: unconnected-(U1-Pad19) -> /MOSI
- U1 pad 20: unconnected-(U1-Pad20) -> /SCK
- U1 pad 21: unconnected-(U1-Pad21) -> /MISO
- U1 pad 28: unconnected-(U1-Pad28) -> /M1_ref_3V
- U1 pad 29: unconnected-(U1-Pad29) -> /M2_ref_3V
- U1 pad 30: unconnected-(U1-Pad30) -> /M3_ref_3V
- U1 pad 31: unconnected-(U1-Pad31) -> /M4_ref_3V
- U1 pad 4: unconnected-(U1-Pad4) -> /bat_level
- U1 pad 5: unconnected-(U1-Pad5) -> /CSN
- U1 pad 6: unconnected-(U1-Pad6) -> /CE
- U1 pad 7: unconnected-(U1-Pad7) -> /Volume_pot
- U1 pad 8: unconnected-(U1-Pad8) -> /Servo
- U3 pad 1: /v_i_msr_M1 -> GNDREF
- U3 pad 2: GNDREF -> +5V
- U3 pad 3: Net-(R1_M1-Pad1) -> VCC
- U4 pad 3: unconnected-(U4-Pad3) -> /CE
- U4 pad 4: unconnected-(U4-Pad4) -> /CSN
- U4 pad 5: unconnected-(U4-Pad5) -> /SCK
- U4 pad 6: unconnected-(U4-Pad6) -> /MOSI
- U4 pad 7: unconnected-(U4-Pad7) -> /MISO
- U_M1 pad 2: unconnected-(U_M1-Pad2) -> /M1_1
- U_M1 pad 3: unconnected-(U_M1-Pad3) -> /M1_2
- U_M1 pad 5: +3V3 -> VCC
Other:
- board size 53.2 x 104.1 mm -> 53.2 x 98.4 mm

Commit message: FC control board V1.0
As ordered from JLC
Parts:
- removed BZ1: Buzzer1, Buzzer_Beeper:Buzzer_12x9.5RM7.6
- removed BZ2: Buzzer2, Buzzer_Beeper:Buzzer_12x9.5RM7.6
- removed BZ3: Buzzer3, Buzzer_Beeper:Buzzer_12x9.5RM7.6
- removed U4: NRF24L01_Breakout, RF_Module:nRF24L01_Breakout
- removed U_M1: TB67H451AFNG,EL, Package_SO:HSOP-8-1EP_3.9x4.9mm_P1.27mm_EP2.41x3.1mm
- removed Volume1: R_Buzzer, Potentiometer_THT:Potentiometer_Alps_RK09K_Single_Horizontal
- added C1: C, Capacitor_SMD:C_1206_3216Metric, F.Cu at (212.5, 160.6)
- added C10: C_Small, Capacitor_SMD:C_0603_1608Metric, F.Cu at (213.1, 146.3)
- added C11: 10µ, Capacitor_SMD:C_0805_2012Metric_Pad1.18x1.45mm_HandSolder, F.Cu at (219.0, 161.7)
- added C12: 10µ, Capacitor_SMD:C_0805_2012Metric_Pad1.18x1.45mm_HandSolder, F.Cu at (219.0, 141.4)
- added C13: 10µ, Capacitor_SMD:C_0805_2012Metric_Pad1.18x1.45mm_HandSolder, F.Cu at (189.2, 141.4)
- added C14: 10µ, Capacitor_SMD:C_0805_2012Metric_Pad1.18x1.45mm_HandSolder, F.Cu at (189.2, 161.7)
- added G***: LOGO, LOGO, F.Cu at (196.2, 107.1)
- added J2: Conn_01x04_Pin, Connector_PinSocket_2.54mm:PinSocket_1x04_P2.54mm_Vertical, F.Cu at (213.0, 185.5)
- added J3: Conn_01x03_Pin, Connector_PinSocket_2.54mm:PinSocket_1x03_P2.54mm_Vertical, F.Cu at (188.9, 183.0)
- added JP1: SolderJumper_3_Bridged12, Jumper:SolderJumper-3_P1.3mm_Bridged12_RoundedPad1.0x1.5mm, B.Cu at (212.5, 147.6)
- added M1: Motor_DC_ALT, Connector_JST:JST_EH_B2B-EH-A_1x02_P2.50mm_Vertical, F.Cu at (220.3, 137.0)
- added M2: Motor_DC_ALT, Connector_JST:JST_EH_B2B-EH-A_1x02_P2.50mm_Vertical, F.Cu at (220.3, 157.3)
- added M3: Motor_DC_ALT, Connector_JST:JST_EH_B2B-EH-A_1x02_P2.50mm_Vertical, F.Cu at (190.5, 137.0)
- added M4: Motor_DC_ALT, Connector_JST:JST_EH_B2B-EH-A_1x02_P2.50mm_Vertical, F.Cu at (190.5, 157.3)
- added R5: R_Small, Resistor_SMD:R_0603_1608Metric_Pad0.98x0.95mm_HandSolder, F.Cu at (209.0, 130.4)
- added R6: R_Small, Resistor_SMD:R_0603_1608Metric_Pad0.98x0.95mm_HandSolder, F.Cu at (209.0, 132.6)
- added R_bat1: 80k, Resistor_SMD:R_0805_2012Metric_Pad1.20x1.40mm_HandSolder, F.Cu at (206.4, 162.4)
- added R_bat2: 50k, Resistor_SMD:R_0805_2012Metric_Pad1.20x1.40mm_HandSolder, F.Cu at (206.4, 165.3)
- added Rsense1: R_Small, Resistor_SMD:R_1206_3216Metric, F.Cu at (215.1, 143.7)
- added Rsense2: R_Small, Resistor_SMD:R_1206_3216Metric, F.Cu at (211.8, 150.7)
- added Rsense3: R_Small, Resistor_SMD:R_1206_3216Metric, F.Cu at (201.1, 143.7)
- added Rsense4: R_Small, Resistor_SMD:R_1206_3216Metric, F.Cu at (202.1, 150.7)
- added U10: ZXBM5210, FC_footprint_library:ZXBM5210, F.Cu at (193.0, 144.3)
- added U11: ZXBM5210, FC_footprint_library:ZXBM5210, F.Cu at (193.0, 164.6)
- added U8: ZXBM5210, FC_footprint_library:ZXBM5210, F.Cu at (222.8, 164.6)
- added U9: LM358_DFN, Package_SO:SOIC-8-1EP_3.9x4.9mm_P1.27mm_EP2.514x3.2mm, F.Cu at (207.0, 136.7)
- U5: value LM358DRG3 2_4 -> ZXBM5210; footprint Package_SO:SOIC-8_3.9x4.9mm_P1.27mm -> FC_footprint_library:ZXBM5210
- U6: value LM358DRG3 1_3 -> INA4181A3IPWR; footprint Package_SO:SOIC-8_3.9x4.9mm_P1.27mm -> FC_footprint_library:SOP65P640X120-20N
- moved C4 90.9 mm to (214.0, 195.1), turned to 90 degrees
- moved R4 82.4 mm to (214.0, 191.1), turned to 90 degrees
- moved R1 78.0 mm to (220.4, 171.0)
- moved C6 76.6 mm to (216.3, 127.2), turned to 90 degrees
- moved U5 76.1 mm to (222.8, 144.3)
- moved BT1 74.9 mm to (222.6, 124.0), turned to 90 degrees
- moved C5 72.9 mm to (212.7, 127.2), turned to 90 degrees
- moved C3 67.1 mm to (206.9, 126.4), turned to 90 degrees
- moved C2 63.9 mm to (203.6, 126.4), turned to 90 degrees
- moved U3 60.9 mm to (214.5, 117.9), turned to 90 degrees
- moved U6 60.1 mm to (207.0, 144.3), turned to 180 degrees
- moved C8 59.8 mm to (198.3, 126.5), turned to 90 degrees
- moved C7 55.9 mm to (195.0, 126.5), turned to 90 degrees
- moved U7 51.1 mm to (196.7, 117.8), turned to 90 degrees
- moved U1 33.3 mm to (202.1, 184.7), turned to 180 degrees
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Connections:
- net /SS renamed /ACD1_9
- U1 pad 12: /SDA -> /ACD1_7
- U1 pad 15: unconnected-(U1-IO3-Pad15) -> /M3_sense
- U1 pad 17: /SCL -> /ACD1_8
- U1 pad 19: /MOSI -> unconnected-(U1-IO11-Pad19)
- U1 pad 20: /SCK -> unconnected-(U1-IO12-Pad20)
- U1 pad 28: /M1_ref_3V -> /FWR_1
- U1 pad 29: /M2_ref_3V -> /REV_1
- U1 pad 30: /M3_ref_3V -> /FWR_2
- U1 pad 31: /M4_ref_3V -> /REV_2
- U1 pad 32: unconnected-(U1-IO39-Pad32) -> /FWR_3
- U1 pad 33: unconnected-(U1-IO40-Pad33) -> /REV_3
- U1 pad 34: unconnected-(U1-IO41-Pad34) -> /FWR_4
- U1 pad 35: unconnected-(U1-IO42-Pad35) -> /REV_4
- U1 pad 38: unconnected-(U1-IO2-Pad38) -> /M2_sense
- U1 pad 39: unconnected-(U1-IO1-Pad39) -> /M1_sense
- U1 pad 4: /bat_level -> /M4_sense
- U1 pad 5: /CSN -> /ACD1_4
- U1 pad 6: /CE -> /ACD1_5
- U1 pad 7: /Volume_pot -> /ACD1_6
- U5 pad 1: /M2_ref_5V -> Net-(M1-+)
- U5 pad 2: Net-(U5A--) -> VCC
- U5 pad 3: /M2_ref_3V -> VCC
- U5 pad 4: GNDREF -> /FWR_2
- U5 pad 5: /M3_ref_3V -> /REV_2
- U5 pad 6: Net-(U5B--) -> VCC
- U5 pad 7: /M3_ref_5V -> /in-2
- U5 pad 8: VCC -> GNDREF
- U6 pad 1: /M4_ref_5V -> Net-(U6-REF1)
- U6 pad 2: Net-(U6A--) -> /M1_sense
- U6 pad 3: /M4_ref_3V -> /in-1
- U6 pad 4: GNDREF -> /in+1
- U6 pad 5: /M1_ref_3V -> Net-(U6-VS)
- U6 pad 6: Net-(U6B--) -> /in+2
- U6 pad 7: /M1_ref_5V -> /in-2
- U6 pad 8: VCC -> /M2_sense
Routing:
- net VCC: track 0.00 -> 189.3 mm, vias 0 -> 19
- net +5V: track 0.00 -> 164.0 mm, vias 0 -> 7
- net +3V3: track 0.00 -> 120.9 mm, vias 0 -> 7
- net GNDREF: track 0.00 -> 71.3 mm, vias 0 -> 29
- net /REV_2: track 0.00 -> 71.3 mm, vias 0 -> 2
- net /M2_sense: track 0.00 -> 67.5 mm, vias 0 -> 4
- net /FWR_2: track 0.00 -> 65.3 mm, vias 0 -> 2
- net /M1_sense: track 0.00 -> 59.0 mm, vias 0 -> 2
- net /REV_3: track 0.00 -> 49.0 mm
- net /IO0: track 0.00 -> 46.9 mm
- net /REV_1: track 0.00 -> 44.4 mm, vias 0 -> 2
- net /M4_sense: track 0.00 -> 43.8 mm
- net /M3_sense: track 0.00 -> 40.3 mm, vias 0 -> 2
- net /FWR_3: track 0.00 -> 39.7 mm
- net /FWR_1: track 0.00 -> 37.5 mm, vias 0 -> 2
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- added copper zone on B.Cu, net GNDREF
Other:
- board text added: "FC Control board v0.1 J. Wheeler G. Abrahamsson 2023"
