File: Steering wheel/Electronics/FC_Wheel_PCB/FC_Wheel_PCB/FC_Wheel_PCB.kicad_pcb (KiCad board)
At the start: 2 copper layers, 124.4 x 77.9 mm, 39 parts, among them J1 USB_C_Receptacle_USB2.0, J2 Display_con, J3 MPU6050_con, SW10 RotaryEncoder_Switch, SW3 SW_SPST, U2 ESP32-S3-WROOM-1-N8, U6 AZ1117-3.3, U7 AZ1117-3.3

Commit message: Finish up wheel PCB
Parts:
- removed BZ3: Buzzer3, Buzzer_Beeper:Buzzer_12x9.5RM7.6
- removed REF**: KiCad-Logo2_5mm_SilkScreen, Symbol:KiCad-Logo2_5mm_SilkScreen
- added J4: L_TRIGGER, Connector_PinHeader_2.54mm:PinHeader_1x03_P2.54mm_Vertical, F.Cu at (187.3, 105.8)
- added J5: R_TRIGGER, Connector_PinHeader_2.54mm:PinHeader_1x03_P2.54mm_Vertical, F.Cu at (73.0, 103.3)
- added PADDLE1: SW_R, Connector_PinHeader_2.00mm:PinHeader_1x02_P2.00mm_Vertical, F.Cu at (107.5, 123.0)
- added PADDLE2: SW_L, Connector_PinHeader_2.00mm:PinHeader_1x02_P2.00mm_Vertical, F.Cu at (148.6, 123.0)
- added R3: 5k, Resistor_SMD:R_0805_2012Metric_Pad1.20x1.40mm_HandSolder, F.Cu at (106.4, 132.5)
- added R4: 50k, Resistor_SMD:R_0805_2012Metric_Pad1.20x1.40mm_HandSolder, F.Cu at (110.9, 132.5)
Connections:
- U2 pad 10: /ENC_A -> /L_TRIGGER
- U2 pad 11: /ENC_B -> /R_TRIGGER
- U2 pad 24: unconnected-(U2-IO47-Pad24) -> /ENC_A
- U2 pad 25: unconnected-(U2-IO48-Pad25) -> /ENC_B
- U2 pad 31: unconnected-(U2-IO38-Pad31) -> /R_PADDLE
- U2 pad 32: unconnected-(U2-IO39-Pad32) -> /L_PADDLE
- U2 pad 35: /BUZZER_PIN3 -> unconnected-(U2-IO42-Pad35)
Routing:
- net +3V0: track 0.00 -> 181.3 mm, vias 0 -> 1
- net /L_TRIGGER: track 0.00 -> 77.1 mm, vias 0 -> 2
- net /R_TRIGGER: track 0.00 -> 65.7 mm, vias 0 -> 2
- net Earth: track 347.7 -> 400.7 mm, vias 10 -> 14
- net /R_PADDLE: track 0.00 -> 47.0 mm, vias 0 -> 1
- net +3V3: track 330.6 -> 371.0 mm, vias 5 -> 6
- net /L_PADDLE: track 0.00 -> 28.5 mm, vias 0 -> 1
- net /BUZZER_PIN3: track 25.1 -> 0.00 mm, vias 1 -> 0
- net /ENC_B: track 41.9 -> 60.2 mm
- net /ENC_A: track 40.3 -> 55.7 mm
- net /BTN6: track 66.6 -> 65.6 mm
- net Net-(BT1--): track 76.6 -> 76.0 mm

Commit message: Polish Wheel PCB [ Ordered ]
Parts:
- added J6: Pinout, Connector_PinHeader_2.54mm:PinHeader_1x07_P2.54mm_Vertical, F.Cu at (156.3, 91.8)
- added REF**: ESD-Logo_6.6x6mm_SilkScreen, Symbol:ESD-Logo_6.6x6mm_SilkScreen, F.Cu at (178.5, 92.5)
- added REF**: OSHW-Logo2_7.3x6mm_SilkScreen, Symbol:OSHW-Logo2_7.3x6mm_SilkScreen, F.Cu at (82.5, 93.0)
- added REF**: KiCad-Logo2_6mm_SilkScreen, Symbol:KiCad-Logo2_6mm_SilkScreen, F.Cu at (108.0, 96.0)
- added REF**: WEEE-Logo_8.4x12mm_SilkScreen, Symbol:WEEE-Logo_8.4x12mm_SilkScreen, B.Cu at (130.5, 102.5)
- SW3: value SW_SPST -> BATTERY_SW
Connections:
- U2 pad 22: unconnected-(U2-IO14-Pad22) -> /IO14
- U2 pad 35: unconnected-(U2-IO42-Pad35) -> /IO42
Routing:
- net /IO14: track 0.00 -> 29.5 mm
- net /IO42: track 0.00 -> 17.7 mm, vias 0 -> 1
- net /SDA: track 55.1 -> 69.2 mm, vias 0 -> 2
- net /SCL: track 43.0 -> 53.2 mm, vias 0 -> 2
- net VCC: track 104.2 -> 113.8 mm
- net Earth: track 400.7 -> 408.9 mm
- net +3V3: track 371.0 -> 375.3 mm
- net /L_TRIGGER: track 77.1 -> 78.9 mm
- net /L_PADDLE: track 28.5 -> 29.5 mm
- net /MISO: track 55.3 -> 54.5 mm
- net /SCK: track 50.3 -> 51.1 mm
Other:
- board text added: "*"
- board text added: "3V3"
- board text added: "GND"
- board text added: "IN"
- board text added: "IO14"
- board text added: "IO42"
- board text added: "MISO"
- board text added: "MOSI"
- board text added: "SCK"
- board text added: "SCL"
- board text added: "SDA"
- board text added: "VCC"
