File: Steering wheel/Electronics/FC_Wheel_PCB/FC_Wheel_PCB/FC_Wheel_PCB.kicad_sch (KiCad schematic)
At the start: 36 parts, among them J1 USB_C_Receptacle_USB2.0, J2 Display_con, J3 MPU6050_con, SW3 RotaryEncoder_Switch, SW3 SW_SPST, U2 ESP32-S3-WROOM-1-N8, U6 AZ1117-3.3, U7 AZ1117-3.3

Commit message: Finish up wheel PCB
Parts:
- removed BZ3: Buzzer3, Buzzer_Beeper:Buzzer_12x9.5RM7.6, symbol Device:Buzzer
- added J4: L_TRIGGER, Connector_PinHeader_2.54mm:PinHeader_1x03_P2.54mm_Vertical, symbol Connector:Conn_01x03_Pin
- added J5: R_TRIGGER, Connector_PinHeader_2.54mm:PinHeader_1x03_P2.54mm_Vertical, symbol Connector:Conn_01x03_Pin
- added PADDLE1: SW_R, Connector_PinHeader_2.00mm:PinHeader_1x02_P2.00mm_Vertical, symbol Switch:SW_SPST
- added PADDLE2: SW_L, Connector_PinHeader_2.00mm:PinHeader_1x02_P2.00mm_Vertical, symbol Switch:SW_SPST
- added R3: 5k, Resistor_SMD:R_0805_2012Metric_Pad1.20x1.40mm_HandSolder, symbol Device:R
- added R4: 50k, Resistor_SMD:R_0805_2012Metric_Pad1.20x1.40mm_HandSolder, symbol Device:R
Connections:
- net +3V3: now also PADDLE1.1 (A), PADDLE2.1 (A), R3.1
- net ENC_A: now also U2.24 (IO47); no longer U2.10 (IO17)
- net ENC_B: now also U2.25 (IO48); no longer U2.11 (IO18)
- net Earth: now also J4.1 (Pin_1), J5.1 (Pin_1), R4.2
- net R_PADDLE: now reaches U2.31 (IO38)
- net R_PADDLE: now also PADDLE1.2 (B)
- net L_PADDLE: now reaches U2.32 (IO39)
- net L_PADDLE: now also PADDLE2.2 (B)
- net BUZZER_PIN3: no longer names the net of U2.35 (IO42)
- new net +3V0: J4.3 (Pin_3), J5.3 (Pin_3), R3.2, R4.1
- new net L_TRIGGER: J4.2 (Pin_2), U2.10 (IO17)
- new net R_TRIGGER: J5.2 (Pin_2), U2.11 (IO18)
Other:
- note added: "3.0V for analog read"
- note added: "Paddles"
- note added: "Triggers (might have to be 3.3V if hall effect sensors are to be used)"
- moved on the sheet: BT1, C2, C8, R10, R11, R12, SW3, U2

Commit message: Polish Wheel PCB [ Ordered ]
Parts:
- added J6: Pinout, Connector_PinHeader_2.54mm:PinHeader_1x07_P2.54mm_Vertical, symbol Connector:Conn_01x07_Pin
- SW3: value SW_SPST -> BATTERY_SW
Connections:
- net +3V3: now also J6.2 (Pin_2)
- net Earth: now also J6.1 (Pin_1)
- net SCL: now also J6.7 (Pin_7)
- net SDA: now also J6.6 (Pin_6)
- net VCC: now also J6.3 (Pin_3)
- net IO14: now reaches U2.22 (IO14)
- net IO14: now also J6.5 (Pin_5)
- net IO42: now reaches U2.35 (IO42)
- net IO42: now also J6.4 (Pin_4)
Other:
- note added: "GPIO"
- note added: "I2C"
- note added: "Miscellaneous pinout"
Changed lines of the file:
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@@
     (stroke (width 0) (type default))
   )
+  (wire (pts (xy 373.38 147.32) (xy 377.19 147.32))
+    (stroke (width 0) (type default))
+  )
   (wire (pts (xy 154.94 128.27) (xy 165.1 128.27))
     (stroke (width 0) (type default))
@@
     (stroke (width 0) (type default))
   )
+  (wire (pts (xy 369.57 142.24) (xy 377.19 142.24))
+    (stroke (width 0) (type default))
+  )
   (wire (pts (xy 250.19 69.85) (xy 254 69.85))
     (stroke (width 0) (type default))
@@
     (stroke (width 0) (type default))
   )
+  (wire (pts (xy 205.74 158.75) (xy 207.01 158.75))
+    (stroke (width 0) (type default))
+  )
   (wire (pts (xy 161.29 26.67) (xy 177.8 26.67))
     (stroke (width 0) (type default))
@@
     (stroke (width 0) (type default))
   )
+  (polyline (pts (xy 346.71 162.56) (xy 407.67 162.56))
+    (stroke (width 0) (type default))
+  )
+  (polyline (pts (xy 406.4 162.56) (xy 406.4 125.73))
+    (stroke (width 0) (type default))
+  )
   (wire (pts (xy 303.53 60.96) (xy 306.07 60.96))
     (stroke (width 0) (type default))
@@
     (stroke (width 0) (type default))
   )
+  (wire (pts (xy 205.74 125.73) (xy 208.28 125.73))
+    (stroke (width 0) (type default))
+  )
   (wire (pts (xy 210.82 102.87) (xy 210.82 106.68))
     (stroke (width 0) (type default))
@@
     (stroke (width 0) (type default))
   )
+  (wire (pts (xy 368.3 139.7) (xy 377.19 139.7))
+    (stroke (width 0) (type default))
+  )
   (wire (pts (xy 375.92 107.95) (xy 375.92 109.22))
     (stroke (width 0) (type default))
@@
     (stroke (width 0) (type default))
   )
+  (wire (pts (xy 369.57 144.78) (xy 377.19 144.78))
+    (stroke (width 0) (type default))
+  )
   (wire (pts (xy 391.16 36.83) (xy 391.16 39.37))
     (stroke (width 0) (type default))
@@
     (stroke (width 0) (type default))
   )
+  (wire (pts (xy 368.3 137.16) (xy 377.19 137.16))
+    (stroke (width 0) (type default))
+  )
   (wire (pts (xy 306.07 74.93) (xy 306.07 77.47))
     (stroke (width 0) (type default))
@@
     (stroke (width 0) (type default))
   )
+  (wire (pts (xy 373.38 149.86) (xy 377.19 149.86))
+    (stroke (width 0) (type default))
+  )
   (wire (pts (xy 307.34 144.78) (xy 307.34 146.05))
     (stroke (width 0) (type default))
@@
     (stroke (width 0) (type default))
   )
+  (wire (pts (xy 373.38 152.4) (xy 377.19 152.4))
+    (stroke (width 0) (type default))
+  )
   (wire (pts (xy 154.94 118.11) (xy 165.1 118.11))
     (stroke (width 0) (type default))
@@
     (stroke (width 0) (type default))
   )
-  (wire (pts (xy 205.74 161.29) (xy 210.82 161.29))
+  (wire (pts (xy 205.74 161.29) (xy 209.55 161.29))
     (stroke (width 0) (type default))
   )
@@
     (effects (font (size 1.27 1.27)) (justify left bottom))
   )
+  (text "I2C\n" (at 364.2091 139.0736 0)
+    (effects (font (size 1.27 1.27)) (justify left bottom))
+  )
+  (text "Miscellaneous pinout" (at 349.25 129.54 0)
+    (effects (font (size 1.27 1.27)) (justify left bottom))
+  )
   (text "USB port" (at 347.98 17.78 0)
     (effects (font (size 1.27 1.27)) (justify left bottom))
@@
     (effects (font (size 1.27 1.27)) (justify left bottom))
   )
+  (text "GPIO\n" (at 364.1031 143.6766 0)
+    (effects (font (size 1.27 1.27)) (justify left bottom))
+  )
+  (label "IO14" (at 369.57 142.24 0) (fields_autoplaced)
+    (effects (font (size 1.27 1.27)) (justify left bottom))
+  )
   (label "ENC_SW" (at 49.53 31.75 0) (fields_autoplaced)
     (effects (font (size 1.27 1.27)) (justify left bottom))
@@
     (effects (font (size 1.27 1.27)) (justify left bottom))
   )
+  (label "SDA" (at 368.3 139.7 0) (fields_autoplaced)
+    (effects (font (size 1.27 1.27)) (justify left bottom))
+  )
   (label "BTN1" (at 154.94 118.11 0) (fields_autoplaced)
     (effects (font (size 1.27 1.27)) (justify left bottom))
@@
     (effects (font (size 1.27 1.27)) (justify left bottom))
   )
-  (label "MISO" (at 210.82 161.29 0) (fields_autoplaced)
+  (label "MISO" (at 209.55 161.29 0) (fields_autoplaced)
     (effects (font (size 1.27 1.27)) (justify left bottom))
   )
@@
     (effects (font (size 1.27 1.27)) (justify left bottom))
   )
+  (label "IO14" (at 207.01 158.75 0) (fields_autoplaced)
+    (effects (font (size 1.27 1.27)) (justify left bottom))
+  )
   (label "BTN2" (at 154.94 120.65 0) (fields_autoplaced)
     (effects (font (size 1.27 1.27)) (justify left bottom))
   )
+  (label "IO42" (at 369.57 144.78 0) (fields_autoplaced)
+    (effects (font (size 1.27 1.27)) (justify left bottom))
+  )
   (label "BTN6" (at 218.44 80.01 0) (fields_autoplaced)
     (effects (font (size 1.27 1.27)) (justify left bottom))
@@
     (effects (font (size 1.27 1.27)) (justify left bottom))
   )
+  (label "SCL" (at 368.3 137.16 0) (fields_autoplaced)
+    (effects (font (size 1.27 1.27)) (justify left bottom))
+  )
   (label "BTN5" (at 218.44 68.58 0) (fields_autoplaced)
     (effects (font (size 1.27 1.27)) (justify left bottom))
@@
     (effects (font (size 1.27 1.27)) (justify left bottom))
   )
+  (label "IO42" (at 208.28 125.73 0) (fields_autoplaced)
+    (effects (font (size 1.27 1.27)) (justify left bottom))
+  )
   (label "ENC_B" (at 54.61 50.8 0) (fields_autoplaced)
     (effects (font (size 1.27 1.27)) (justify left bottom))
@@
     )
   )
+  (symbol (lib_id "Connector:Conn_01x07_Pin") (at 382.27 144.78 180) (unit 1)
+    (in_bom yes) (on_board yes) (dnp no) (fields_autoplaced)
+    (property "Reference" "J6" (at 383.54 143.51 0)
+      (effects (font (size 1.27 1.27)) (justify right))
+    )
+    (property "Value" "Pinout" (at 383.54 146.05 0)
+      (effects (font (size 1.27 1.27)) (justify right))
+    )
+    (property "Footprint" "Connector_PinHeader_2.54mm:PinHeader_1x07_P2.54mm_Vertical" (at 382.27 144.78 0)
+      (effects (font (size 1.27 1.27)) hide)
+    )
+    (property "Datasheet" "~" (at 382.27 144.78 0)
+      (effects (font (size 1.27 1.27)) hide)
+    )
+    (pin "1")
+    (pin "2")
+    (pin "3")
+    (pin "4")
+    (pin "5")
+    (pin "6")
+    (pin "7")
+    (instances
+      (project "FC_Wheel_PCB"
+        (path "/c6386384-eee7-4d8e-abab-84cc9b6b83e0"
+          (reference "J6") (unit 1)
+        )
+      )
+    )
+  )
   (symbol (lib_id "power:VCC") (at 375.92 96.52 0) (unit 1)
     (in_bom yes) (on_board yes) (dnp no) (fields_autoplaced)
@@
       (effects (font (size 1.27 1.27)) (justify right))
     )
-    (property "Value" "SW_SPST" (at 377.19 115.57 90)
+    (property "Value" "BATTERY_SW" (at 377.19 115.57 90)
       (effects (font (size 1.27 1.27)) (justify right))
     )
@@
     )
   )
+  (symbol (lib_id "power:+3V3") (at 373.38 149.86 90) (unit 1)
+    (in_bom yes) (on_board yes) (dnp no) (fields_autoplaced)
+    (property "Reference" "#PWR057" (at 377.19 149.86 0)
+      (effects (font (size 1.27 1.27)) hide)
+    )
+    (property "Value" "+3V3" (at 369.57 149.86 90)
+      (effects (font (size 1.27 1.27)) (justify left))
+    )
+    (property "Footprint" "" (at 373.38 149.86 0)
+      (effects (font (size 1.27 1.27)) hide)
+    )
+    (property "Datasheet" "" (at 373.38 149.86 0)
+      (effects (font (size 1.27 1.27)) hide)
+    )
+    (pin "1")
+    (instances
+      (project "FC_Wheel_PCB"
+        (path "/c6386384-eee7-4d8e-abab-84cc9b6b83e0"
+          (reference "#PWR057") (unit 1)
+        )
+      )
+      (project "FC Control board 1.0"
+        (path "/e63e39d7-6ac0-4ffd-8aa3-1841a4541b55"
+          (reference "#PWR0119") (unit 1)
+        )
+      )
+    )
+  )
   (symbol (lib_id "power:+3V3") (at 243.84 102.87 90) (unit 1)
     (in_bom yes) (on_board yes) (dnp no) (fields_autoplaced)
@@
     )
   )
+  (symbol (lib_id "power:VCC") (at 373.38 147.32 90) (unit 1)
+    (in_bom yes) (on_board yes) (dnp no) (fields_autoplaced)
+    (property "Reference" "#PWR056" (at 377.19 147.32 0)
+      (effects (font (size 1.27 1.27)) hide)
+    )
+    (property "Value" "VCC" (at 369.57 147.32 90)
+      (effects (font (size 1.27 1.27)) (justify left))
+    )
+    (property "Footprint" "" (at 373.38 147.32 0)
+      (effects (font (size 1.27 1.27)) hide)
+    )
+    (property "Datasheet" "" (at 373.38 147.32 0)
+      (effects (font (size 1.27 1.27)) hide)
+    )
+    (pin "1")
+    (instances
+      (project "FC_Wheel_PCB"
+        (path "/c6386384-eee7-4d8e-abab-84cc9b6b83e0"
+          (reference "#PWR056") (unit 1)
+        )
+      )
+      (project "FC Control board 1.0"
+        (path "/e63e39d7-6ac0-4ffd-8aa3-1841a4541b55"
+          (reference "#PWR0122") (unit 1)
+        )
+      )
+    )
+  )
   (symbol (lib_name "+3V3_1") (lib_id "power:+3V3") (at 77.47 31.75 0) (unit 1)
     (in_bom yes) (on_board yes) (dnp no) (fields_autoplaced)
@@
         )
       )
+    )
+  )
+  (symbol (lib_id "power:Earth") (at 373.38 152.4 0) (unit 1)
+    (in_bom yes) (on_board yes) (dnp no) (fields_autoplaced)
+    (property "Reference" "#PWR055" (at 373.38 158.75 0)
+      (effects (font (size 1.27 1.27)) hide)
+    )
+    (property "Value" "Earth" (at 373.38 156.21 0)
+      (effects (font (size 1.27 1.27)) hide)
+    )
+    (property "Footprint" "" (at 373.38 152.4 0)
+      (effects (font (size 1.27 1.27)) hide)
+    )
+    (property "Datasheet" "~" (at 373.38 152.4 0)
+      (effects (font (size 1.27 1.27)) hide)
+    )
+    (pin "1")
+    (instances
+      (project "FC_Wheel_PCB"
+        (path "/c6386384-eee7-4d8e-abab-84cc9b6b83e0"
+          (reference "#PWR055") (unit 1)
+        )
+      )
