File: Steering wheel/Electronics/16_Channel_LED_Strip/16_Channel_LED_Strip/16_Channel_LED_Strip.kicad_pcb (KiCad board)
At the start: 2 copper layers, 91 x 31.4 mm, 38 parts, among them IC1 TLC59116FIPWR, J1 INPUT

Commit message: Finish LED PCB [Ordered]
Parts:
- removed REF**: ESD-Logo_6.6x6mm_SilkScreen, Symbol:ESD-Logo_6.6x6mm_SilkScreen
- moved R3 17.8 mm to (144.0, 99.2)
- moved R1 6.10 mm to (156.0, 99.2)
- moved R2 6.10 mm to (149.9, 99.2)
- moved R0 6.10 mm to (162.0, 99.2)
- moved R_I2C_1 5.49 mm to (120.7, 115.2)
- moved R_I2C_2 5.14 mm to (120.6, 109.7)
- moved R4 0.12 mm to (155.9, 104.2)
- moved R5 0.12 mm to (149.9, 104.2)
- moved R6 0.12 mm to (143.9, 104.2)
Routing:
- net +BATT: track 0.00 -> 106.6 mm
- net Net-(D0-K): track 0.00 -> 57.2 mm, vias 0 -> 1
- net Earth: track 0.00 -> 54.8 mm, vias 0 -> 1
- net Net-(D1-K): track 0.00 -> 50.9 mm, vias 0 -> 1
- net Net-(D2-K): track 0.00 -> 44.5 mm, vias 0 -> 1
- net Net-(D14-K): track 0.00 -> 40.9 mm, vias 0 -> 1
- net +3V3: track 0.00 -> 40.2 mm, vias 0 -> 2
- net Net-(D3-K): track 0.00 -> 38.3 mm, vias 0 -> 1
- net Net-(D13-K): track 0.00 -> 34.7 mm, vias 0 -> 1
- net Net-(D4-K): track 0.00 -> 33.5 mm, vias 0 -> 1
- net Net-(D12-K): track 0.00 -> 28.6 mm, vias 0 -> 1
- net Net-(D5-K): track 0.00 -> 25.4 mm, vias 0 -> 1
- net Net-(D11-K): track 0.00 -> 21.9 mm, vias 0 -> 1
- net Net-(D5-A): track 0.00 -> 21.5 mm
- net Net-(D2-A): track 0.00 -> 21.0 mm
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- added copper zone on F.Cu, net +BATT
- added copper zone on B.Cu, net Earth
Other:
- board text removed: "FC_Wheel 1.0 2023"
