File: Steering wheel/Electronics/FC_Wheel_PCB/FC_Wheel_PCB-2.0/FC_Wheel_PCB-2.0.kicad_pcb (KiCad board)
At the start: 2 copper layers, 166.8 x 90.3 mm, 47 parts, among them J1 USB_C_Receptacle_USB2.0, J2 Display_con, J3 MPU6050_con, J4 L_TRIGGER, J5 R_TRIGGER, J6 Pinout, J7 LED_Driver, SW10 RotaryEncoder_Switch, SW3 BATTERY_SW, U2 ESP32-S3-WROOM-1-N8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

Commit message: FC_Wheel_PCB 2.0 [Ordered]
Parts:
- added G***: LOGO, LOGO, F.Cu at (266.5, 188.8)
- added G***: LOGO, LOGO, F.Cu at (278.8, 183.2)
- added REF**: KiCad-Logo2_6mm_SilkScreen, Symbol:KiCad-Logo2_6mm_SilkScreen, F.Cu at (216.0, 133.2)
- added REF**: WEEE-Logo_8.4x12mm_SilkScreen, Symbol:WEEE-Logo_8.4x12mm_SilkScreen, B.Cu at (216.8, 184.8)
- added REF**: ESD-Logo_6.6x6mm_SilkScreen, Symbol:ESD-Logo_6.6x6mm_SilkScreen, F.Cu at (165.2, 137.0)
- added REF**: OSHW-Logo2_7.3x6mm_SilkScreen, Symbol:OSHW-Logo2_7.3x6mm_SilkScreen, F.Cu at (278.5, 151.5)
- J1: value USB_C_Receptacle_USB2.0 -> USB_C
- SW10: value RotaryEncoder_Switch -> RotaryEncoder
- moved R2 6.39 mm to (178.0, 152.5)
- moved U2 6.35 mm to (169.3, 117.4)
- moved C5 4.69 mm to (201.4, 116.7)
- moved R12 4.65 mm to (212.2, 119.2)
- moved U7 4.36 mm to (265.9, 175.8)
- moved R_bat2 4.27 mm to (195.9, 125.4)
- moved R11 4.04 mm to (216.4, 119.2)
- moved R10 1.15 mm to (154.2, 125.9)
- moved C8 1.05 mm to (154.9, 113.5)
- moved C2 1.01 mm to (155.0, 119.4)
Connections:
- J2 pad 5: unconnected-(J2-Pin_5-Pad5) -> /RST
- J2 pad 6: unconnected-(J2-Pin_6-Pad6) -> /DC
- U2 pad 8: unconnected-(U2-IO15-Pad8) -> /DC
- U2 pad 9: unconnected-(U2-IO16-Pad9) -> /RST
Routing:
- net Earth: track 0.00 -> 470.1 mm, vias 0 -> 10
- net +3V3: track 0.00 -> 436.5 mm, vias 0 -> 11
- net /SCL: track 0.00 -> 181.8 mm, vias 0 -> 1
- net /SDA: track 0.00 -> 177.3 mm, vias 0 -> 1
- net /BTN4: track 0.00 -> 137.5 mm, vias 0 -> 2
- net /R_TRIGGER: track 0.00 -> 137.5 mm, vias 0 -> 1
- net VCC: track 0.00 -> 135.8 mm, vias 0 -> 1
- net /BTN3: track 0.00 -> 134.6 mm, vias 0 -> 2
- net Net-(BT1--): track 0.00 -> 120.6 mm
- net /BUZZER_PIN2: track 0.00 -> 110.7 mm, vias 0 -> 2
- net /R_PADDLE: track 0.00 -> 95.7 mm, vias 0 -> 3
- net /Volume_pot: track 0.00 -> 93.1 mm, vias 0 -> 2
- net /ENC_SW: track 0.00 -> 80.1 mm, vias 0 -> 1
- net /EN: track 0.00 -> 79.0 mm, vias 0 -> 1
- net /LED_RESET: track 0.00 -> 75.5 mm, vias 0 -> 1
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- added copper zone on F.Cu, net +3V3
- added copper zone on B.Cu, net Earth
Other:
- outline, holes or cut-outs redrawn
- board text added: "* * * * SDA SCL GND 3V3"
- board text added: "3V3"
- board text added: "BOOT"
- board text added: "FC_Wheel 2.0 2023"
- board text added: "G. Abrahamsson"
- board text added: "GND"
- board text added: "GND 3V3 SCK"
- board text added: "GND 3V3 VCC * IO14 SDA SCL"
- board text added: "GND IN 3V3"
- board text added: "IN"
- board text added: "J. Wheeler"
- board text added: "MOSI RST DC * MISO"
- board text added: "RESET"
- board text added: "RST SDA SCL VCC 3V3 GND"
- board text removed: "3V3 VCC * IO14 SDA SCL"
- board text removed: "GND IN 3V0"
