File: Steering wheel/Electronics/FC_Wheel_PCB/FC_Wheel_PCB-2.0/FC_Wheel_PCB-2.0.kicad_sch (KiCad schematic)
At the start: 39 parts, among them J1 USB_C_Receptacle_USB2.0, J2 Display_con, J3 MPU6050_con, J4 L_TRIGGER, J5 R_TRIGGER, J6 Pinout, J7 LED_Driver, SW3 BATTERY_SW, SW3 RotaryEncoder_Switch, U2 ESP32-S3-WROOM-1-N8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

Commit message: FC_Wheel_PCB 2.0 [Ordered]
Connections:
- net RST: now reaches J2.5 (Pin_5)
- net RST: now also U2.9 (IO16)
- net DC: now reaches J2.6 (Pin_6)
- net DC: now also U2.8 (IO15)
- no-connect marks 2 -> 16
Other:
- moved on the sheet: BZ1, BZ2, C8, R10, S1, S3, Volume1
