File: Electronics/PCB/FC Control board 1.3/FC Control board 1.3.kicad_pcb (KiCad board)
At the start: 2 copper layers, 53.2 x 98.4 mm, 49 parts, among them IC1 A3909GLNTR-T, IC2 A3909GLNTR-T, J1 USB_C_Receptacle_USB2.0, J2 CAM, J3 Servo, J4 Hall-M1, J5 Hall-M2, J6 Hall-M0, J7 Hall-M3, M3 Motor_DC_ALT, SW1 RST, SW2 BOOT, SW3 PWR_SW, U1 ESP32-S3-WROOM-1-N8, U10 ZXBM5210, U2 AZ1117-3.3, U3 AZ1117-5.0, U6 INA4181A3IPWR, U7 AZ1117-3.3, U9 LM358_DFN

Commit message: Continue FC 1.3
Parts:
- removed Rsense3: R_Small, Resistor_SMD:R_1206_3216Metric
- removed SW3: PWR_SW, Connector_PinHeader_2.00mm:PinHeader_1x02_P2.00mm_Vertical
- removed U10: ZXBM5210, FC_footprint_library:ZXBM5210
- added ADR0: ADR_BIT, Jumper:SolderJumper-3_P1.3mm_Open_RoundedPad1.0x1.5mm_NumberLabels, F.Cu at (201.6, 154.5)
- added C11: C_MAYBE, Capacitor_SMD:C_1206_3216Metric, F.Cu at (214.9, 114.8)
- added C12: 47uF, Capacitor_SMD:CP_Elec_6.3x5.4, F.Cu at (196.3, 110.3)
- added C14: 47uF, Capacitor_SMD:CP_Elec_6.3x5.4, F.Cu at (217.0, 110.3)
- added C15: 47uF, Capacitor_SMD:CP_Elec_6.3x5.4, F.Cu at (213.1, 139.7)
- added C16: 47uF, Capacitor_SMD:CP_Elec_6.3x5.4, F.Cu at (206.6, 126.7)
- added C17: C_MAYBE, Capacitor_SMD:C_1206_3216Metric, F.Cu at (199.2, 147.2)
- added C18: C_MAYBE, Capacitor_SMD:C_1206_3216Metric, F.Cu at (213.6, 147.0)
- added C19: 47uF, Capacitor_SMD:CP_Elec_6.3x5.4, F.Cu at (200.1, 139.7)
- added C21: 100n, Capacitor_SMD:C_0805_2012Metric_Pad1.18x1.45mm_HandSolder, F.Cu at (209.6, 152.8)
- added C9: C_MAYBE, Capacitor_SMD:C_1206_3216Metric, F.Cu at (198.3, 114.8)
- added D3: CUHS20S30,H3F, FC_footprint_library:CUHS20S30,H3F, F.Cu at (195.7, 130.5)
- added D4: CUHS20S30,H3F, FC_footprint_library:CUHS20S30,H3F, F.Cu at (219.2, 124.3)
- added D5: BAT_LED, LED_SMD:LED_0805_2012Metric_Pad1.15x1.40mm_HandSolder, F.Cu at (219.0, 137.6)
- added D6: CUHS20S30,H3F, FC_footprint_library:CUHS20S30,H3F, F.Cu at (203.4, 131.9)
- added F2: PPTC 500mA, Fuse:Fuse_1206_3216Metric, F.Cu at (219.6, 182.7)
- added M0: Motor_DC_ALT, Connector_JST:JST_EH_B2B-EH-A_1x02_P2.50mm_Vertical, F.Cu at (191.4, 105.5)
- added M1: Motor_DC_ALT, Connector_JST:JST_EH_B2B-EH-A_1x02_P2.50mm_Vertical, F.Cu at (219.6, 104.5)
- added M2: Motor_DC_ALT, Connector_JST:JST_EH_B2B-EH-A_1x02_P2.50mm_Vertical, F.Cu at (193.9, 151.2)
- added Q1: SQ2348ES-T1_BE3, Package_TO_SOT_SMD:SOT-23-3, F.Cu at (224.0, 116.2)
- added R10: 2K, Resistor_SMD:R_0603_1608Metric_Pad0.98x0.95mm_HandSolder, F.Cu at (218.9, 143.5)
- added R11: 10K, Resistor_SMD:R_0603_1608Metric_Pad0.98x0.95mm_HandSolder, F.Cu at (218.9, 140.7)
- added R12: 10K, Resistor_SMD:R_0603_1608Metric_Pad0.98x0.95mm_HandSolder, F.Cu at (202.1, 165.7)
- added R13: 10K, Resistor_SMD:R_0603_1608Metric_Pad0.98x0.95mm_HandSolder, F.Cu at (202.1, 168.7)
- added R8: 100K, Resistor_SMD:R_0603_1608Metric_Pad0.98x0.95mm_HandSolder, F.Cu at (220.6, 117.2)
- added R9: 1K, Resistor_SMD:R_0603_1608Metric_Pad0.98x0.95mm_HandSolder, F.Cu at (219.0, 134.6)
- added R_S1: 0.01, Resistor_SMD:R_1206_3216Metric, F.Cu at (210.9, 112.8)
- added R_S2: 0.01, Resistor_SMD:R_1206_3216Metric, F.Cu at (193.1, 141.2)
- added R_S3: 0.01, Resistor_SMD:R_1206_3216Metric, F.Cu at (213.6, 150.7)
- added SW4: ~, FC_footprint_library:LSS12-P-V-B, F.Cu at (223.9, 141.0)
- added U8: LSM6DSM (LSM6DSMTR), FC_footprint_library:LSM6DSM, F.Cu at (206.6, 155.2)
- C13: value 10µ -> 100n
- R1, R2, R3, R4, R7: footprint Resistor_SMD:R_0805_2012Metric_Pad1.20x1.40mm_HandSolder -> Resistor_SMD:R_0603_1608Metric_Pad0.98x0.95mm_HandSolder
- U1: footprint RF_Module:ESP32-S3-WROOM-1 -> FC_footprint_library:ESP32-S3-WROOM-1-N8
- U2, U7: value AZ1117-3.3 -> AZ1117IH-3.3TRG1
- U3: value AZ1117-5.0 -> AZ1117D-5.0TRE1
- moved R_S0 77.0 mm to (202.4, 112.8), turned to 90 degrees
- moved R5 71.3 mm to (280.1, 125.5)
- moved R6 71.3 mm to (280.1, 127.6)
- moved C10 70.1 mm to (282.2, 135.0)
- moved U6 70.1 mm to (276.1, 133.0)
- moved U9 70.1 mm to (276.1, 125.3)
- moved M3 64.4 mm to (219.1, 148.7), turned to -90 degrees
- moved J6 64.1 mm to (199.9, 101.8), turned to -64.5 degrees
- moved J7 62.5 mm to (225.1, 172.0)
- moved U4 61.0 mm to (206.6, 118.7)
- moved IC1 57.7 mm to (206.6, 109.7), turned to 90 degrees
- moved G*** 57.5 mm to (195.1, 163.4)
- moved C13 53.2 mm to (203.6, 158.1), turned to 0 degrees
- moved U5 51.7 mm to (206.6, 148.7)
- moved IC2 43.5 mm to (206.6, 139.7), turned to 90 degrees
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- renumbered R_S1 to R_S0
Connections:
- BT1 pad 2: unconnected-(BT1---Pad2) -> Net-(BT1--)
- C13 pad 1: Net-(M3-+) -> GNDREF
- C13 pad 2: /in-3 -> +3V3
- C2 pad 2: VCC -> Net-(D4-K)
- C5 pad 2: VCC -> Net-(D3-K)
- C7 pad 2: +5V -> Net-(D6-K)
- IC1 pad 1: unconnected-(IC1-IN1-Pad1) -> /M0_A
- IC1 pad 10: unconnected-(IC1-OUT1-Pad10) -> Net-(IC1-OUT1)
- IC1 pad 2: unconnected-(IC1-IN2-Pad2) -> /M0_B
- IC1 pad 3: unconnected-(IC1-VBB-Pad3) -> VCC
- IC1 pad 4: unconnected-(IC1-IN3-Pad4) -> /M1_A
- IC1 pad 5: unconnected-(IC1-IN4-Pad5) -> /M1_B
- IC1 pad 6: unconnected-(IC1-OUT4-Pad6) -> /in-1
- IC1 pad 7: unconnected-(IC1-OUT3-Pad7) -> Net-(IC1-OUT3)
- IC1 pad 8: unconnected-(IC1-GND-Pad8) -> GNDREF
- IC1 pad 9: unconnected-(IC1-OUT2-Pad9) -> /in-0
- IC2 pad 1: unconnected-(IC2-IN1-Pad1) -> /M2_A
- IC2 pad 10: unconnected-(IC2-OUT1-Pad10) -> Net-(IC2-OUT1)
- IC2 pad 2: unconnected-(IC2-IN2-Pad2) -> /M2_B
- IC2 pad 3: unconnected-(IC2-VBB-Pad3) -> VCC
- IC2 pad 4: unconnected-(IC2-IN3-Pad4) -> /M3_A
- IC2 pad 5: unconnected-(IC2-IN4-Pad5) -> /M3_B
- IC2 pad 6: unconnected-(IC2-OUT4-Pad6) -> /in-3
- IC2 pad 7: unconnected-(IC2-OUT3-Pad7) -> Net-(IC2-OUT3)
- IC2 pad 8: unconnected-(IC2-GND-Pad8) -> GNDREF
- IC2 pad 9: unconnected-(IC2-OUT2-Pad9) -> /in-2
- J1 pad A4: +5V -> Net-(F2-Pad1)
- J1 pad A9: +5V -> Net-(F2-Pad1)
- J1 pad B4: +5V -> Net-(F2-Pad1)
- J1 pad B9: +5V -> Net-(F2-Pad1)
- M3 pad 1: Net-(M3-+) -> Net-(IC2-OUT3)
- R_S0 pad 1: unconnected-(R_S1-Pad1) -> /in+0
- R_S0 pad 2: unconnected-(R_S1-Pad2) -> /in-0
- U1 pad 10: unconnected-(U1-IO17-Pad10) -> /M2_sense
- U1 pad 11: unconnected-(U1-IO18-Pad11) -> /M3_sense
- U1 pad 12: /Hall_effect_4 -> /SDA
- U1 pad 15: /M3_sense -> unconnected-(U1-IO3-Pad15)
- U1 pad 17: /ADC1_8 -> /SCL
- U1 pad 18: /ADC1_9 -> /M0_DIR
- U1 pad 19: /BUZZER_PIN -> /M1_DIR
- U1 pad 20: unconnected-(U1-IO12-Pad20) -> /M2_DIR
- U1 pad 21: /TAIL_LED -> /M3_DIR
- U1 pad 22: unconnected-(U1-IO14-Pad22) -> /FWR_0
- U1 pad 23: unconnected-(U1-IO21-Pad23) -> /bat_level
- U1 pad 28: /FWR_1 -> /TAIL_LED
- U1 pad 29: /REV_1 -> /REV_0
- U1 pad 30: /FWR_2 -> /FWR_1
- U1 pad 31: /REV_2 -> /REV_1
- U1 pad 32: /FWR_3 -> /FWR_2
- U1 pad 33: /REV_3 -> /REV_2
- U1 pad 34: /FWR_4 -> /FWR_3
- U1 pad 35: /REV_4 -> /REV_3
- U1 pad 38: /M2_sense -> /BUZZER_PIN
- U1 pad 39: /M1_sense -> /Servo
- U1 pad 4: /M4_sense -> /Hall_effect_0
- U1 pad 8: /Servo -> /M0_sense
- U1 pad 9: unconnected-(U1-IO16-Pad9) -> /M1_sense
- U2 pad 3: VCC -> Net-(D4-K)
- U3 pad 3: VCC -> Net-(D3-K)
- U4 pad 1: Net-(U4-1Y1) -> /M0_B
- U4 pad 11: Net-(U4-3Y0) -> /M1_A
- U4 pad 13: Net-(U4-3Y0) -> /M1_A
- U4 pad 15: Net-(U4-3Y1) -> /M1_B
- U4 pad 3: Net-(U4-1Y0) -> /M0_A
- U4 pad 5: Net-(U4-1Y0) -> /M0_A
- U4 pad 7: Net-(U4-1Y1) -> /M0_B
- U4 pad 9: Net-(U4-3Y1) -> /M1_B
- U5 pad 1: Net-(U5-1Y1) -> /M2_B
- U5 pad 11: Net-(U5-3Y0) -> /M3_A
- U5 pad 13: Net-(U5-3Y0) -> /M3_A
- U5 pad 15: Net-(U5-3Y1) -> /M3_B
- U5 pad 3: Net-(U5-1Y0) -> /M2_A
- U5 pad 5: Net-(U5-1Y0) -> /M2_A
- U5 pad 7: Net-(U5-1Y1) -> /M2_B
- U5 pad 9: Net-(U5-3Y1) -> /M3_B
- U7 pad 3: +5V -> Net-(D6-K)
Routing:
- net /Hall_effect_0: track 0.00 -> 105.6 mm, vias 0 -> 1
- net /Servo: track 0.00 -> 94.8 mm, vias 0 -> 1
- net +5V: track 0.00 -> 88.7 mm, vias 0 -> 5
- net /Hall_effect_1: track 0.00 -> 88.6 mm, vias 0 -> 1
- net /REV_1: track 0.00 -> 76.2 mm, vias 0 -> 2
- net /FWR_1: track 0.00 -> 71.8 mm, vias 0 -> 2
- net /REV_0: track 0.00 -> 66.0 mm, vias 0 -> 2
- net /USB_VBUS: track 0.00 -> 65.3 mm, vias 0 -> 6
- net /M1_DIR: track 0.00 -> 64.9 mm, vias 0 -> 2
- net /FWR_0: track 0.00 -> 63.7 mm, vias 0 -> 2
- net /M0_DIR: track 0.00 -> 59.9 mm, vias 0 -> 2
- net /EN: track 0.00 -> 51.9 mm, vias 0 -> 4
- net /REV_3: track 0.00 -> 50.0 mm, vias 0 -> 2
- net /FWR_3: track 0.00 -> 44.3 mm, vias 0 -> 2
- net /FWR_2: track 0.00 -> 42.1 mm, vias 0 -> 2
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- added copper zone on F.Cu, net +3V3
Other:
- board text added: "2S LiPo"
- board text added: "FC Control board v1.3 G. Abrahamsson J. Wheeler 2023"
- board text added: "GND +3V3 IN"
- board text removed: "ESP32-S3-WROOM-1"
- board text removed: "FC Control board v1.2 J. Wheeler G. Abrahamsson 2023"
- board text removed: "GND +3V3 SENS"
- board text removed: "Servo"
