File: Electronics/PCB/FC Control board 1.3/FC Control board 1.3.kicad_sch (KiCad schematic)
At the start: 44 parts, among them IC1 A3909GLNTR-T, IC2 A3909GLNTR-T, J1 USB_C_Receptacle_USB2.0, J2 CAM, J3 Servo, J4 Hall-M1, J5 Hall-M2, J6 Hall-M0, J7 Hall-M3, SW1 RST, SW2 BOOT, SW3 PWR_SW, U1 ESP32-S3-WROOM-1-N8, U2 AZ1117-3.3, U4 AZ1117-5.0, U6 INA4181A3IPWR, U7 AZ1117-3.3, U9 LM358_DFN

Commit message: Continue FC 1.3
Parts:
- removed SW3: PWR_SW, Connector_PinHeader_2.00mm:PinHeader_1x02_P2.00mm_Vertical, symbol Switch:SW_SPST
- added ADR0: ADR_BIT, Jumper:SolderJumper-3_P1.3mm_Open_RoundedPad1.0x1.5mm_NumberLabels, symbol Jumper:SolderJumper_3_Open
- added C11, C17, C18, C9: C_MAYBE, Capacitor_SMD:C_1206_3216Metric, symbol Device:C_Small
- added C12, C14, C15, C16, C19: 47uF, Capacitor_SMD:CP_Elec_6.3x5.4, symbol Device:C_Polarized
- added C13, C21: 100n, Capacitor_SMD:C_0805_2012Metric_Pad1.18x1.45mm_HandSolder, symbol Device:C_Small
- added D11 (x3): CUHS20S30,H3F, FC_footprint_library:CUHS20S30,H3F, symbol Device:D_Schottky
- added D5: BAT_LED, LED_SMD:LED_0805_2012Metric_Pad1.15x1.40mm_HandSolder, symbol Device:LED
- added F1: PPTC 500mA, Fuse:Fuse_1206_3216Metric, symbol Device:Fuse_Small
- added M0, M1, M2, M3: Motor_DC_ALT, Connector_JST:JST_EH_B2B-EH-A_1x02_P2.50mm_Vertical, symbol Motor:Motor_DC_ALT
- added Q1: SQ2348ES-T1_BE3, Package_TO_SOT_SMD:SOT-23-3, symbol Transistor_FET:IRLZ24
- added R10: 2K, Resistor_SMD:R_0603_1608Metric_Pad0.98x0.95mm_HandSolder, symbol Device:R_Small
- added R11, R12, R13: 10K, Resistor_SMD:R_0603_1608Metric_Pad0.98x0.95mm_HandSolder, symbol Device:R
- added R8: 100K, Resistor_SMD:R_0603_1608Metric_Pad0.98x0.95mm_HandSolder, symbol Device:R
- added R9: 1K, Resistor_SMD:R_0603_1608Metric_Pad0.98x0.95mm_HandSolder, symbol Device:R
- added R_S1, R_S2, R_S3: 0.01, Resistor_SMD:R_1206_3216Metric, symbol Device:R_Small
- added SW4: ~, FC_footprint_library:LSS12-P-V-B, symbol FC_library:LSS12-P-V-B
- added U8: LSM6DSM (LSM6DSMTR), FC_footprint_library:LSM6DSM, symbol Sensor_Motion:LSM6DSM
- IC1, IC2: footprint SOP100P600X175-10N -> FC_footprint_library:SOP100P600X175-10N
- R1, R2, R3, R4, R7: footprint Resistor_SMD:R_0805_2012Metric_Pad1.20x1.40mm_HandSolder -> Resistor_SMD:R_0603_1608Metric_Pad0.98x0.95mm_HandSolder
- U1: footprint ESP32-S3-WROOM-1-N8_EXP -> FC_footprint_library:ESP32-S3-WROOM-1-N8
- U2, U7: value AZ1117-3.3 -> AZ1117IH-3.3TRG1
- U4: value AZ1117-5.0 -> AZ1117D-5.0TRE1
- renumbered R_S1 to R_S0
Connections:
- net +3V3: now also ADR0.3 (B), C13.2, C21.2, R12.1, R13.1, U8.12 (CS), U8.5 (VDDIO), U8.8 (VDD)
- net +5V: now also C19.1; no longer C7.2, J1.A4 (VBUS), J1.A9 (VBUS), J1.B4 (VBUS), J1.B9 (VBUS), U7.3 (VI)
- net GNDREF: now also IC1.8 (GND), IC2.8 (GND), ADR0.1 (A), C12.2, C13.1, C14.2, C15.2, C16.2, C19.2, C21.1, Q1.2 (S), R10.1, R11.2, R8.2, U8.2 (SDX), U8.3 (SCX), U8.6 (GND), U8.7 (GND)
- net SCL: now also R13.2, U8.13 (SCL)
- net SDA: now also R12.2, U8.14 (SDA)
- net VCC: now also IC1.3 (VBB), IC2.3 (VBB), C12.1, C14.1, C15.1, C16.1, D11.2 (A), D11.2 (A), SW4.1 (A); no longer C2.2, C7.2, U2.3 (VI), U4.3 (VI)
- net in+0: now also R_S0.1, M0.2 (-)
- net in+1: now also M1.2 (-), R_S1.1
- net in+2: now also M2.2 (-), R_S2.1
- net in+3: now also M3.2 (-), R_S3.1
- net in-0: now also IC1.9 (OUT2), R_S0.2, C9.1
- net in-1: now also IC1.6 (OUT4), C11.1, R_S1.2
- net in-2: now also IC2.9 (OUT2), C17.1, R_S2.2
- net in-3: now also IC2.6 (OUT4), C18.1, R_S3.2
- net M2_A: now reaches IC2.1 (IN1)
- net M2_A: now also U5.3 (1Y0), U5.5 (2Y1)
- net at IC2.10 (OUT1): now also C17.2, M2.1 (+)
- net M2_B: now reaches IC2.2 (IN2)
- net M2_B: now also U5.1 (1Y1), U5.7 (2Y0)
- net M3_A: now reaches IC2.4 (IN3)
- net M3_A: now also U5.11 (3Y0), U5.13 (4Y1)
- net M3_B: now reaches IC2.5 (IN4)
- net M3_B: now also U5.15 (4Y0), U5.9 (3Y1)
- net at IC2.7 (OUT3): now also C18.2, M3.1 (+)
- net at BT1.2 (-): now also Q1.3 (D)
- net M0_A: now reaches IC1.1 (IN1)
- net M0_A: now also U4.3 (1Y0), U4.5 (2Y1)
- net at IC1.10 (OUT1): now also C9.2, M0.1 (+)
- net M0_B: now reaches IC1.2 (IN2)
- net M0_B: now also U4.1 (1Y1), U4.7 (2Y0)
- net M1_A: now reaches IC1.4 (IN3)
- net M1_A: now also U4.11 (3Y0), U4.13 (4Y1)
- net M1_B: now reaches IC1.5 (IN4)
- net M1_B: now also U4.15 (4Y0), U4.9 (3Y1)
- net at IC1.7 (OUT3): now also C11.2, M1.1 (+)
- new net: C7.2, D11.1 (K), U7.3 (VI)
- new net: D5.1 (K), R10.2
- new net: D5.2 (A), R9.1, SW4.2 (COM)
- new net: ADR0.2 (C), U8.1 (SDO/SA0)
- new net: C7.2, D11.1 (K), U4.3 (VI)
- new net: Q1.1 (G), R8.1, R9.2
- new net: F1.1, J1.A4 (VBUS), J1.A9 (VBUS), J1.B4 (VBUS), J1.B9 (VBUS)
- new net: C2.2, D11.1 (K), U2.3 (VI)
- new net: R11.1, SW4.3 (B)
- new net USB_VBUS: D11.2 (A), F1.2
- no-connect marks 10 -> 14
Other:
- removed sheet Motor driver2
- note added: ""MODE 1": HOST<->IMU through SPI/I2C I2C Enabled: CS = 1 * THIS IS USED * SPI Enabled: CS = 0"
- note added: "500mA (h) fuse: 0ZCJ0050AF2E"
- note added: "Battery and MOSFET with switch"
- note added: "Capacitors: EEV476M035S9GAA"
- note added: "Hall effect sensors for the wheels: DRV5056A2QLPGM"
- note added: "I2C Pullup resistors"
- note added: "IMU"
- note added: "Motor control"
- note removed: "Hall effect sensors for the wheels"
- moved on the sheet: BT1, C2, IC1, IC2, R_S0
